Commit message: dd

File: mybot_description/urdf/mybot.xacro (robot description, xacro)
@@ -6,7 +6,7 @@
 <xacro:property name="chassisLength" value="0.4"/>
 <xacro:property name="chassisWidth" value="0.2"/>
-<xacro:property name="chassisMass" value="2"/>
+<xacro:property name="chassisMass" value="5"/>
 <xacro:property name="casterRadius" value="0.05"/>
-<xacro:property name="casterMass" value="2"/>
+<xacro:property name="casterMass" value="3"/>
 <xacro:property name="wheelWidth" value="0.05"/>
 <xacro:property name="wheelRadius" value="0.1"/>
